Commit message: Update GUI with simulation model

File: medsnake_description/urdf/medsnake.xacro (robot description, xacro)
@@ -21,5 +21,5 @@
   <xacro:property name="link_radius" value="0.005405" />
   <xacro:property name="link_length" value="0.00923" />
-  <xacro:property name="num_links" value="30" />
+  <xacro:property name="num_links" value="20" />
   <xacro:property name="first_length" value="0.15" />
   <xacro:property name="first_radius" value="0.00923" />
@@ -50,5 +50,5 @@
     <parent link="base_link" />
     <child link="link_inner" />
-    <origin rpy="1.5707963 0 1.5707963" xyz="0.1 0 0.04" />
+    <origin rpy="1.5707963 0 1.5707963" xyz="0.01 0 0.04" />
     <limit effort="1000" lower="0" upper="0.35000000000000003" velocity="180" />
     <axis xyz="0 0 1" />
@@ -82,5 +82,5 @@
     <parent link="base_link" />
     <child link="link_outer" />
-    <origin rpy="1.5707963 0 1.5707963" xyz="0.2 0 0.04" />
+    <origin rpy="1.5707963 0 1.5707963" xyz="0.08 0 0.04" />
     <limit effort="1000" lower="0" upper="0.35000000000000003" velocity="180" />
     <axis xyz="0 0 1" />
@@ -228,16 +228,14 @@
   </xacro:macro>
   <xacro:loop num_links="${num_links}" />
+<!--
   <joint name="camera_joint" type="fixed">
     <parent link="link_30" />
     <child link="camera_link" />
     <origin rpy="-1.570796 -1.570796 0" xyz="0 0 0" />
-    <!-- <axis xyz="0 0 1" /> -->
+    <axis xyz="0 0 1" />
   </joint>
   <link name="camera_link">
     <xacro:default_inertial mass="0.001"/>
     <visual>
-      <!-- <geometry>
-        <cylinder length="0.1" radius="0.001" />
-      </geometry> -->
       <material name="red"/>
       <origin rpy="0 0 0" xyz="0 0 0" />
@@ -263,7 +261,4 @@
         <noise>
           <type>gaussian</type>
-          <!-- Noise is sampled independently per pixel on each frame.
-               That pixel's noise value is added to each of its color
-               channels, which at that point lie in the range [0,1]. -->
           <mean>0.0</mean>
           <stddev>0.007</stddev>
@@ -285,5 +280,5 @@
       </plugin>
     </sensor>
-  </gazebo>
+  </gazebo> -->
   <!-- <link name = "link_snake">
     <inertial>
